Commit message: update map

File: install/my_bot/share/my_bot/description/agv.urdf.xacro (robot description, xacro)
@@ -1,207 +1 @@
-<?xml version="1.0"?>
-<robot xmlns:xacro="http://www.ros.org/wiki/xacro" name="my_bot">
-    <!-- base_footprint -->
-    <link name="base_footprint"/>
-    <!-- base_link -->
- <link
-    name="base_link">
-    <inertial>
-      <origin
-        xyz="-1.1536E-16 -8.6736E-17 0.13512"
-        rpy="0 0 0" />
-      <mass
-        value="201.67" />
-      <inertia
-        ixx="9.5313"
-        ixy="-9.2157E-16"
-        ixz="-5.6579E-16"
-        iyy="22.658"
-        iyz="-4.198E-17"
-        izz="30.077" />
-    </inertial>
-    <visual>
-      <origin
-        xyz="0 0 0"
-        rpy="0 0 0" />
-      <geometry>
-            <mesh filename="file://$(find my_bot)/meshes/base_link.STL"/>
-      </geometry>
-      <material
-        name="">
-        <color
-          rgba="0.79216 0.81961 0.93333 1" />
-      </material>
-    </visual>
-    <collision>
-      <origin
-        xyz="0 0 0"
-        rpy="0 0 0" />
-      <geometry>
-            <mesh filename="file://$(find my_bot)/meshes/base_link.STL"/>
-      </geometry>
-    </collision>
-  </link>
-    <!-- base_footprint -> base_link joint -->
-    <joint name="base_footprint_joint" type="fixed">
-        <origin xyz="0 0 0" rpy="0 0 0"/>
-        <parent link="base_footprint"/>
-        <child link="base_link"/>
-    </joint>
-   <link
-    name="left_wheel">
-    <inertial>
-      <origin
-        xyz="6.0715E-18 -0.02 0"
-        rpy="0 0 0" />
-      <mass
-        value="0.80425" />
-      <inertia
-        ixx="0.001394"
-        ixy="6.1901E-35"
-        ixz="7.1778E-51"
-        iyy="0.0025736"
-        iyz="2.4867E-36"
-        izz="0.001394" />
-    </inertial>
-    <visual>
-      <origin
-        xyz="0 0 0"
-        rpy="0 0 0" />
-      <geometry>
-        <mesh filename="file://$(find my_bot)/meshes/left_wheel.STL"/>
-      </geometry>
-      <material
-        name="">
-        <color
-          rgba="0.79216 0.81961 0.93333 1" />
-      </material>
-    </visual>
-    <collision>
-      <origin
-        xyz="0 0 0"
-        rpy="0 0 0" />
-      <geometry>
-        <mesh filename="file://$(find my_bot)/meshes/left_wheel.STL"/>
-      </geometry>
-    </collision>
-  </link>
-  <joint
-    name="leftwheel"
-    type="continuous">
-    <origin
-      xyz="0 0.406 0.018995"
-      rpy="0 0 0" />
-    <parent
-      link="base_link" />
-    <child
-      link="left_wheel" />
-    <axis
-      xyz="0 1 0" />
-    <dynamics
-      friction="0.1" />
-  </joint>
-    <link
-    name="right_wheel">
-    <inertial>
-      <origin
-        xyz="6.9389E-18 0.02 0"
-        rpy="0 0 0" />
-      <mass
-        value="0.80425" />
-      <inertia
-        ixx="0.001394"
-        ixy="6.1901E-35"
-        ixz="7.1778E-51"
-        iyy="0.0025736"
-        iyz="2.4867E-36"
-        izz="0.001394" />
-    </inertial>
-    <visual>
-      <origin
-        xyz="0 0 0"
-        rpy="0 0 0" />
-      <geometry>
-        <mesh filename="file://$(find my_bot)/meshes/right_wheel.STL"/>
-      </geometry>
-      <material
-        name="">
-        <color
-          rgba="0.79216 0.81961 0.93333 1" />
-      </material>
-    </visual>
-    <collision>
-      <origin
-        xyz="0 0 0"
-        rpy="0 0 0" />
-      <geometry>
-        <mesh filename="file://$(find my_bot)/meshes/right_wheel.STL"/>
-      </geometry>
-    </collision>
-  </link>
-  <joint
-    name="rightwheel"
-    type="continuous">
-    <origin
-      xyz="0 -0.406 0.018995"
-      rpy="0 0 0" />
-    <parent
-      link="base_link" />
-    <child
-      link="right_wheel" />
-    <axis
-      xyz="0 1 0" />
-    <dynamics
-      friction="0.1" />
-  </joint>
-    <link
-    name="lidar_link">
-    <inertial>
-      <origin
-        xyz="-8.6736E-18 0 -0.02"
-        rpy="0 0 0" />
-      <mass
-        value="0.45239" />
-      <inertia
-        ixx="0.00046747"
-        ixy="0"
-        ixz="-1.4694E-36"
-        iyy="0.00046747"
-        iyz="-1.0491E-36"
-        izz="0.0008143" />
-    </inertial>
-    <visual>
-      <origin
-        xyz="0 0 0"
-        rpy="0 0 0" />
-      <geometry>
-        <mesh filename="file://$(find my_bot)/meshes/lidar_link.STL"/>
-      </geometry>
-      <material
-        name="">
-        <color
-          rgba="0.79216 0.81961 0.93333 1" />
-      </material>
-    </visual>
-    <collision>
-      <origin
-        xyz="0 0 0"
-        rpy="0 0 0" />
-      <geometry>
-        <mesh filename="file://$(find my_bot)/meshes/lidar_link.STL"/>
-      </geometry>
-    </collision>
-  </link>
-  <joint
-    name="lidar_joint"
-    type="fixed">
-    <origin
-      xyz="0 0 0.29909"
-      rpy="0 0 0" />
-    <parent
-      link="base_link" />
-    <child
-      link="lidar_link" />
-    <axis
-      xyz="0 0 1" />
-  </joint>
-</robot>
+/home/ender/Desktop/dev_ws/src/my_bot/description/agv.urdf.xacro

File: install/my_bot/share/my_bot/description/gazebo_control.xacro (robot description, xacro)
@@ -1,79 +1 @@
-<?xml version="1.0" ?>
-<robot xmlns:xacro="http://www.ros.org/wiki/xacro">
-    <gazebo reference="base_link">
-        <material>Gazebo/Yellow</material>
-    </gazebo>
-    <gazebo reference="left_wheel">
-        <material>Gazebo/Black</material>
-    </gazebo>
-    <gazebo reference="right_wheel">
-        <material>Gazebo/Black</material>
-    </gazebo>
-    <gazebo reference="lidar_link">
-        <material>Gazebo/Orange</material>
-    </gazebo>
-    <gazebo reference="left_back_caster">
-        <material>Gazebo/Black</material>
-    </gazebo>
-    <gazebo reference="right_back_caster">
-        <material>Gazebo/Black</material>
-    </gazebo>
-    <gazebo reference="left_front_caster">
-        <material>Gazebo/Black</material>
-    </gazebo>
-    <gazebo reference="right_front_caster">
-        <material>Gazebo/Black</material>
-    </gazebo>
-    <gazebo>
-      <plugin name="diff_drive" filename="libgazebo_ros_diff_drive.so">
-        <!-- Name of left joint, defaults to `left_joint` -->
-        <left_joint>leftwheel</left_joint>
-        <!-- Name of right joint, defaults to `right_joint` -->
-        <right_joint>rightwheel</right_joint>
-        <!-- The distance from the center of one wheel to the other, in meters, defaults to 0.34 m -->
-        <wheel_separation>0.812</wheel_separation>
-        <!-- Diameter of the wheels, in meters, defaults to 0.15 m -->
-        <wheel_diameter>0.16</wheel_diameter>
-        <!-- Wheel acceleration, in rad/s^2, defaults to 0.0 rad/s^2 -->
-        <max_wheel_acceleration>50.0</max_wheel_acceleration>
-        <!-- Maximum torque which the wheels can produce, in Nm, defaults to 5 Nm -->
-        <max_wheel_torque>200</max_wheel_torque>
-        <!-- Odometry frame, defaults to `odom` -->
-        <odometry_frame>odom</odometry_frame>
-        <!-- Robot frame to calculate odometry from, defaults to `base_footprint` -->
-        <robot_base_frame>base_footprint</robot_base_frame>
-        <!-- Output -->
-        <publish_odom>true</publish_odom>
-        <publish_odom_tf>true</publish_odom_tf>
-        <publish_wheel_tf>true</publish_wheel_tf>
-      </plugin>
-    </gazebo>
-   <!-- hokuyo -->
-  <gazebo reference="lidar_link">
-    <sensor name="front_hokuyo_sensor" type="ray" >
-      <pose>0 0 0 0 0 0</pose>
-      <visualize>false</visualize>
-      <update_rate>10</update_rate>
-      <ray>
-        <scan>
-          <horizontal>
-            <samples>360</samples>
-            <min_angle>-3.14</min_angle>
-            <max_angle>3.14</max_angle>
-          </horizontal>
-        </scan>
-        <range>
-          <min>0.3</min>
-          <max>12.0</max>
-        </range>
-      </ray>
-      <plugin name="gazebo_ros_head_hokuyo_controller" filename="libgazebo_ros_ray_sensor.so">
-          <ros>
-              <argument>~/out:=scan</argument>
-          </ros>
-          <output_type>sensor_msgs/LaserScan</output_type>
-        <frame_name>lidar_link</frame_name>
-      </plugin>
-    </sensor>
-  </gazebo>
-</robot>
+/home/ender/Desktop/dev_ws/src/my_bot/description/gazebo_control.xacro

File: install/my_bot/share/my_bot/description/robot.urdf.xacro (robot description, xacro)
@@ -1,5 +1 @@
-<?xml version="1.0"?>
-<robot xmlns:xacro="http://www.ros.org/wiki/xacro"  name="robot">
-    <xacro:include filename="agv.urdf.xacro" />
-    <xacro:include filename="gazebo_control.xacro" />
-</robot>
+/home/ender/Desktop/dev_ws/src/my_bot/description/robot.urdf.xacro
